File: ZibokPadPCB/ZibokPadPCB.sch (KiCad schematic (older format))
At the start: 14 parts

Commit message: Key schematic finish
Parts:
- added D? (x26): D_Small, symbol Device:D_Small
- added F?: Polyfuse_Small, symbol Device:Polyfuse_Small
- added MX? (x26): MX-NoLED, symbol MX_Alps_Hybrid:MX-NoLED
- added USB?: Molex-0548190589, symbol random-keyboard-parts:Molex-0548190589
Connections:
- net labels added: COL0, COL1, COL2, COL3, ROW0, ROW1, ROW2, ROW3, ROW4, VCC
- wire segments 44 -> 123

Commit message: Continuation
Parts:
- added SW2: Rotary_Encoder, Rotary_Encoder:RotaryEncoder_Alps_EC11E-Switch_Vertical_H20mm, symbol Device:Rotary_Encoder
- C1, C2, C3, C4, C5, C6, C7: renamed from C?; footprint (none) -> Capacitor_SMD:C_0805_2012Metric
- D1, D10, D11, D12, D13, D14, D15, D16, D17, D18, D19, D2, D20, D21, D22, D23, D24, D25, D26, D3, D4, D5, D6, D7, D8, D9: renamed from D?; footprint (none) -> Diode_SMD:D_SOD-123
- F1: renamed from F?; footprint (none) -> Fuse:Fuse_1206_3216Metric
- MX1, MX2, MX25, MX26: renamed from MX?; footprint (none) -> MX_Only:MXOnly-2U-NoLED
- MX10, MX11, MX12, MX13, MX14, MX15, MX16, MX17, MX18, MX20, MX21, MX22, MX23, MX24, MX3, MX4, MX5, MX6, MX7, MX9: renamed from MX?; footprint (none) -> MX_Only:MXOnly-1U-NoLED
- MX19, MX8: renamed from MX?; footprint (none) -> MX_Only:MXOnly-2U-ReversedStabilizers-NoLED
- R1, R2, R3, R4: renamed from R?; footprint (none) -> Resistor_SMD:R_0805_2012Metric
- SW1: renamed from SW?; footprint (none) -> random-keyboard-parts:SKQG-1155865
- USB1: renamed from USB?; footprint (none) -> random-keyboard-parts:Molex-0548190589
- Y1: renamed from Y?; footprint (none) -> Crystal:Crystal_SMD_3225-4Pin_3.2x2.5mm
- gave numbers to parts that had none: 1

Commit message: Switched to stm32
Parts:
- removed D1, D19, D2, D25, D26, D8: D_Small, Diode_SMD:D_SOD-123, symbol Device:D_Small
- removed MX1, MX2, MX25, MX26: MX-NoLED, MX_Only:MXOnly-2U-NoLED, symbol MX_Alps_Hybrid:MX-NoLED
- removed MX19, MX8: MX-NoLED, MX_Only:MXOnly-2U-ReversedStabilizers-NoLED, symbol MX_Alps_Hybrid:MX-NoLED
- removed R2: 22, Resistor_SMD:R_0805_2012Metric, symbol Device:R_Small
- removed R3: R_Small, Resistor_SMD:R_0805_2012Metric, symbol Device:R_Small
- removed R4: 10k, Resistor_SMD:R_0805_2012Metric, symbol Device:R_Small
- removed SW1: SW_Push, random-keyboard-parts:SKQG-1155865, symbol Switch:SW_Push
- removed SW2: Rotary_Encoder, Rotary_Encoder:RotaryEncoder_Alps_EC11E-Switch_Vertical_H20mm, symbol Device:Rotary_Encoder
- removed U1: ATmega32U4-AU, Package_QFP:TQFP-44_10x10mm_P0.8mm, symbol MCU_Microchip_ATmega:ATmega32U4-AU
- removed Y1: Crystal_GND24_Small, Crystal:Crystal_SMD_3225-4Pin_3.2x2.5mm, symbol Device:Crystal_GND24_Small
- added C8: 1uF, symbol Device:C_Small
- added CRST1: 100uF, symbol Device:C_Small
- added CRST2, CS1: 4.7nF, symbol Device:C_Small
- added CUSB1, CVR1, CVR2: 0.1uF, symbol Device:C_Small
- added D1: D_TVS, symbol Device:D_TVS
- added D2: D_Schottky, symbol Device:D_Schottky
- added DRST1: 1N4148, symbol Device:D_Small
- added Q1: DTC123J, symbol Transistor_BJT:DTC123J
- added RRST1: 100k, symbol Device:R_Small
- added RS1: 1M, symbol Device:R_Small
- added RST1: SW_Push, symbol Switch:SW_Push
- added SW?: Rotary_Encoder_Switch, symbol Device:Rotary_Encoder_Switch
- added U1: STM32F072C8Tx, Package_QFP:LQFP-48_7x7mm_P0.5mm, symbol MCU_ST_STM32F0:STM32F072C8Tx
- added U2: USBLC6-2SC6, Package_TO_SOT_SMD:SOT-23-6, symbol Power_Protection:USBLC6-2SC6
- added U3: MCP1700-3302E_SOT23, Package_TO_SOT_SMD:SOT-23, symbol Regulator_Linear:MCP1700-3302E_SOT23
- C1, C4: value 0.1 uF -> 0.1uF; footprint Capacitor_SMD:C_0805_2012Metric -> (none)
- C2, C3: value 12 pF -> 0.1uF; footprint Capacitor_SMD:C_0805_2012Metric -> (none)
- C5: value 0.1 uF -> 4.7uF; footprint Capacitor_SMD:C_0805_2012Metric -> (none)
- C6: value 10 uF -> 4.7uF; footprint Capacitor_SMD:C_0805_2012Metric -> (none)
- C7: value 1uF -> 10nF; footprint Capacitor_SMD:C_0805_2012Metric -> (none)
- F1: footprint Fuse:Fuse_1206_3216Metric -> (none)
- R1: value 22 -> 33k; footprint Resistor_SMD:R_0805_2012Metric -> (none)
Connections:
- net labels added: +3.3V, BOOT0, DBus+, Dbus-, NRST, ROT0, ROT1, ROT2, SWCLK, SWDIO, VBUS
- net labels removed: VCC
- wire segments 123 -> 140
Other:
- moved on the sheet: D10, D11, D12, D13, D14, D15, D16, D17, D18, D20, D21, D22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
