File: ZibokPadPCB/ZibokPadPCB.kicad_pcb (KiCad board)
At the start: 2 copper layers, 69 parts, among them SW1 SW_Push, SW2 Rotary_Encoder, U1 ATmega32U4-AU, Y1 Crystal_GND24_Small

Commit message: Switched to stm32
Parts:
- removed D1, D19, D2, D25, D26, D8: D_Small, Diode_SMD:D_SOD-123
- D10, D11, D12, D13, D14, D15, D16, D17, D18, D20, D21, D22, D23, D24, D3, D4, D5, D6, D7, D9: moved to B.Cu
- moved D3 178.7 mm to (65.3, -104.6), turned to 90 degrees
- moved D14 175.8 mm to (103.4, -104.6), turned to 90 degrees
- moved D9 169.6 mm to (84.3, -104.6), turned to 90 degrees
- moved D20 165.8 mm to (122.6, -104.6), turned to 90 degrees
- moved D21 164.0 mm to (120.3, -85.9), turned to 90 degrees
- moved D4 163.0 mm to (63.1, -85.9), turned to 90 degrees
- moved D10 159.2 mm to (82.2, -85.9), turned to 90 degrees
- moved D15 153.8 mm to (101.2, -85.9), turned to 90 degrees
- moved D5 149.1 mm to (61.5, -66.9), turned to 90 degrees
- moved D11 135.3 mm to (82.2, -66.8), turned to 90 degrees
- moved D16 134.5 mm to (101.1, -66.8), turned to 90 degrees
- moved D22 130.4 mm to (118.2, -66.8), turned to 90 degrees
- moved D6 129.0 mm to (63.1, -47.8), turned to 90 degrees
- moved D23 120.9 mm to (121.5, -47.6), turned to 90 degrees
- moved D17 112.4 mm to (101.1, -47.8), turned to 90 degrees
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Connections:
- MX1 pad 2: Net-(D1-Pad2) -> Net-(D4-Pad2)
- MX19 pad 2: Net-(D19-Pad2) -> Net-(D24-Pad2)
- MX2 pad 2: Net-(D2-Pad2) -> Net-(D6-Pad2)
- MX25 pad 2: Net-(D25-Pad2) -> Net-(D21-Pad2)
- MX26 pad 2: Net-(D26-Pad2) -> Net-(D23-Pad2)
- MX8 pad 2: Net-(D8-Pad2) -> Net-(D13-Pad2)
Routing:
- net COL3: track 0.00 -> 98.3 mm
- net COL1: track 0.00 -> 85.7 mm
- net COL0: track 0.00 -> 84.2 mm
- net COL2: track 0.00 -> 80.3 mm
- net ROW3: track 0.00 -> 59.1 mm
- net ROW0: track 0.00 -> 57.3 mm
- net ROW2: track 0.00 -> 56.8 mm
- net ROW4: track 0.00 -> 45.0 mm
- net ROW1: track 0.00 -> 38.1 mm
- net Net-(D23-Pad2): track 0.00 -> 23.0 mm
- net Net-(D6-Pad2): track 0.00 -> 21.6 mm
- net Net-(D4-Pad2): track 0.00 -> 21.6 mm
- net Net-(D7-Pad2): track 0.00 -> 21.5 mm
- net Net-(D13-Pad2): track 0.00 -> 20.9 mm
- net Net-(D21-Pad2): track 0.00 -> 20.0 mm
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
Commit message: Started routing
Parts:
- removed MX1, MX2, MX25, MX26: MX-NoLED, MX_Only:MXOnly-2U-NoLED
- removed MX19, MX8: MX-NoLED, MX_Only:MXOnly-2U-ReversedStabilizers-NoLED
- removed R2: 22, Resistor_SMD:R_0805_2012Metric
- removed R3: R_Small, Resistor_SMD:R_0805_2012Metric
- removed R4: 10k, Resistor_SMD:R_0805_2012Metric
- removed SW2: Rotary_Encoder, Rotary_Encoder:RotaryEncoder_Alps_EC11E-Switch_Vertical_H20mm
- removed Y1: Crystal_GND24_Small, Crystal:Crystal_SMD_3225-4Pin_3.2x2.5mm
- added C8: 1uF, Capacitor_SMD:C_0805_2012Metric, B.Cu at (22.1, -119.2)
- added CRST1: 100uF, Capacitor_SMD:C_0805_2012Metric, B.Cu at (36.9, -106.2)
- added CRST2: 4.7nF, Capacitor_SMD:C_0805_2012Metric, B.Cu at (32.5, -103.2)
- added CS1: 4.7nF, Capacitor_SMD:C_0805_2012Metric, B.Cu at (31.3, -112.1)
- added CUSB1: 0.1uF, Capacitor_SMD:C_0805_2012Metric, B.Cu at (30.4, -115.8)
- added CVR1: 0.1uF, Capacitor_SMD:C_0805_2012Metric, B.Cu at (36.9, -109.1)
- added CVR2: 0.1uF, Capacitor_SMD:C_0805_2012Metric, B.Cu at (35.7, -112.1)
- added D1: D_TVS, Diode_SMD:D_SOD-123, B.Cu at (21.8, -111.4)
- added D2: D_Schottky, Diode_SMD:D_SOD-123, B.Cu at (12.8, -115.3)
- added DRST1: 1N4148, Diode_SMD:D_SOD-123, B.Cu at (33.1, -100.1)
- added Q1: DTC123J, Package_TO_SOT_SMD:SOT-523, B.Cu at (40.8, -102.9)
- added RRST1: 100k, Resistor_SMD:R_0805_2012Metric, B.Cu at (31.0, -118.7)
- added RS1: 1M, Resistor_SMD:R_0805_2012Metric, B.Cu at (34.8, -115.0)
- added RST1: SW_Push, random-keyboard-parts:SKQG-1155865, B.Cu at (119.0, -124.5)
- added U2: USBLC6-2SC6, Package_TO_SOT_SMD:SOT-23-6, B.Cu at (21.3, -115.4)
- added U3: MCP1700-3302E_SOT23, Package_TO_SOT_SMD:SOT-23, B.Cu at (26.9, -112.0)
- C1, C4: value 0.1 uF -> 0.1uF; moved to B.Cu
- C2, C3: value 12 pF -> 0.1uF; moved to B.Cu
- C5: value 0.1 uF -> 4.7uF; moved to B.Cu
- C6: value 10 uF -> 4.7uF; moved to B.Cu
- C7: value 1uF -> 10nF; moved to B.Cu
- F1, USB1: moved to B.Cu
- R1: value 22 -> 33k; moved to B.Cu
- SW1: value SW_Push -> Rotary_Encoder_Switch; footprint random-keyboard-parts:SKQG-1155865 -> Rotary_Encoder:RotaryEncoder_Alps_EC11E-Switch_Vertical_H20mm
- U1: value ATmega32U4-AU -> STM32F072C8Tx; footprint Package_QFP:TQFP-44_10x10mm_P0.8mm -> Package_QFP:LQFP-48_7x7mm_P0.5mm; moved to B.Cu
- moved F1 218.3 mm to (12.7, -118.7)
- moved C6 214.6 mm to (26.0, -115.8)
- moved C3 213.2 mm to (17.7, -119.2)
- moved C1 211.6 mm to (26.5, -118.7)
- moved C7 209.8 mm to (32.5, -109.1)
- moved USB1 203.0 mm to (70.9, -137.8), turned to 270 degrees
- moved U1 200.9 mm to (109.1, -128.9)
- moved C5 199.6 mm to (32.5, -106.2)
- moved R1 198.3 mm to (40.1, -112.1)
- moved SW1 198.0 mm to (49.7, -131.1)
- moved C4 192.4 mm to (36.9, -103.2)
- moved C2 176.8 mm to (38.2, -99.9)
- moved D24 7.75 mm to (120.1, -28.7)
- moved D7 7.11 mm to (63.1, -28.7)
- moved D20 2.42 mm to (120.1, -104.8)
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Connections:
- net Net-(U1-Pad37) renamed SWCLK
- net VCC renamed VBUS
- C1 pad 1: +5V -> +3V3
- C2 pad 1: Net-(C2-Pad1) -> +3V3
- C3 pad 1: Net-(C3-Pad1) -> +3V3
- C4 pad 1: +5V -> +3V3
- C5 pad 1: +5V -> +3V3
- C6 pad 1: +5V -> +3V3
- C7 pad 1: Net-(C7-Pad1) -> +3V3
- R1 pad 1: Net-(R1-Pad1) -> BOOT0
- R1 pad 2: D- -> Net-(DRST1-Pad1)
- U1 pad 1: Net-(U1-Pad1) -> +3V3
- U1 pad 13: Net-(R3-Pad2) -> Net-(U1-Pad13)
- U1 pad 14: +5V -> Net-(U1-Pad14)
- U1 pad 15: GND -> Net-(U1-Pad15)
- U1 pad 16: Net-(C3-Pad1) -> Net-(U1-Pad16)
- U1 pad 17: Net-(C2-Pad1) -> Net-(U1-Pad17)
- U1 pad 2: +5V -> Net-(U1-Pad2)
- U1 pad 24: +5V -> +3V3
- U1 pad 3: Net-(R1-Pad1) -> Net-(U1-Pad3)
- U1 pad 32: Net-(U1-Pad32) -> D-
- U1 pad 33: Net-(R4-Pad1) -> D+
- U1 pad 34: +5V -> SWDIO
- U1 pad 36: Net-(U1-Pad36) -> +3V3
- U1 pad 43: GND -> Net-(U1-Pad43)
- U1 pad 44: +5V -> BOOT0
- U1 pad 5: GND -> Net-(U1-Pad5)
- U1 pad 6: Net-(C7-Pad1) -> Net-(U1-Pad6)
- U1 pad 7: +5V -> NRST
- U1 pad 8: Net-(U1-Pad8) -> GND
- U1 pad 9: Net-(U1-Pad9) -> +3V3
- USB1 pad 3: D+ -> DBus+
- USB1 pad 4: D- -> Dbus-
Routing:
- net (no net): track 0.00 -> 68.6 mm
- net ROW1: track 38.1 -> 57.2 mm
- net ROW4: track 45.0 -> 57.0 mm
- net Net-(D23-Pad2): track 23.0 -> 11.4 mm
- net COL2: track 80.3 -> 91.7 mm
- net Net-(D6-Pad2): track 21.6 -> 11.4 mm
- net Net-(D4-Pad2): track 21.6 -> 11.4 mm
- net Net-(D7-Pad2): track 21.5 -> 11.4 mm
- net Net-(D13-Pad2): track 20.9 -> 11.4 mm
- net COL0: track 84.2 -> 93.3 mm
- net Net-(D21-Pad2): track 20.0 -> 11.4 mm
- net Net-(D24-Pad2): track 19.5 -> 11.4 mm
- net COL1: track 85.7 -> 93.3 mm
- net COL3: track 98.3 -> 91.7 mm
- net Net-(D22-Pad2): track 8.64 -> 11.4 mm
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
Commit message: routing
Parts:
- moved D2 67.8 mm to (79.2, -128.7)
- moved U2 67.2 mm to (86.7, -130.8), turned to 180 degrees
- moved F1 62.7 mm to (74.9, -126.2), turned to 180 degrees
- moved RRST1 58.5 mm to (89.4, -117.6), turned to 90 degrees
- moved CRST2 55.9 mm to (86.6, -117.0)
- moved CUSB1 55.2 mm to (84.2, -127.9)
- moved U3 54.0 mm to (79.1, -125.6)
- moved DRST1 53.2 mm to (82.9, -118.7), turned to 90 degrees
- moved CRST1 51.6 mm to (87.8, -114.6)
- moved Q1 49.6 mm to (86.9, -121.3)
- moved CVR2 47.7 mm to (82.0, -123.3), turned to 270 degrees
- moved R1 43.8 mm to (83.8, -114.6), turned to 180 degrees
- moved CVR1 41.8 mm to (76.2, -123.3), turned to 270 degrees
- moved U1 7.96 mm to (105.3, -121.9), turned to 90 degrees
Connections:
- CRST2 pad 1: Net-(CRST2-Pad1) -> GND
- U2 pad 1: D- -> D+
- U2 pad 3: D+ -> D-
- U2 pad 4: DBus+ -> Dbus-
- U2 pad 6: Dbus- -> DBus+
Routing:
- net (no net): track 68.6 -> 0.00 mm
- net BOOT0: track 0.00 -> 39.0 mm
- net GND: track 0.00 -> 25.0 mm
- net D+: track 0.00 -> 22.8 mm
- net D-: track 0.00 -> 22.0 mm
- net Dbus-: track 0.00 -> 17.8 mm
- net DBus+: track 0.00 -> 16.8 mm
- net +3V3: track 0.00 -> 9.61 mm
- net +5V: track 0.00 -> 9.57 mm
- net VBUS: track 0.00 -> 7.14 mm
- net NRST: track 0.00 -> 4.33 mm
- net Net-(DRST1-Pad2): track 0.00 -> 3.45 mm
- net Net-(DRST1-Pad1): track 0.00 -> 2.56 mm
Other:
- net class Default: trace_width 0.25 -> 0.254
- net class Power added: clearance 0.2, trace_width 0.381, via_dia 0.8, via_drill 0.4

Commit message: Routing
Parts:
- moved RST1 2.16 mm to (117.5, -122.9)
Connections:
- U1 pad 19: Net-(U1-Pad19) -> COL3
- U1 pad 20: Net-(U1-Pad20) -> COL2
- U1 pad 21: Net-(U1-Pad21) -> COL1
- U1 pad 22: Net-(U1-Pad22) -> COL0
- U1 pad 39: Net-(U1-Pad39) -> ROW4
- U1 pad 40: Net-(U1-Pad40) -> ROW3
- U1 pad 41: Net-(U1-Pad41) -> ROW2
- U1 pad 42: Net-(U1-Pad42) -> ROW1
- U1 pad 43: Net-(U1-Pad43) -> ROW0
Routing:
- net ROW4: track 57.0 -> 169.0 mm
- net ROW3: track 57.2 -> 149.2 mm
- net ROW2: track 57.2 -> 129.0 mm
- net COL0: track 93.3 -> 158.7 mm, vias 0 -> 1
- net ROW1: track 57.2 -> 108.8 mm
- net COL1: track 93.3 -> 130.2 mm, vias 0 -> 1
- net Net-(DRST1-Pad2): track 3.45 -> 38.2 mm, vias 0 -> 2
- net ROW0: track 57.0 -> 88.8 mm
- net COL3: track 91.7 -> 122.8 mm, vias 0 -> 1
- net COL2: track 91.7 -> 110.4 mm, vias 0 -> 1
